File: Schematics/RelativityTimer/RelativityTimer.kicad_pcb (KiCad board)
At the start: 2 copper layers, 11 parts, among them J1 Conn_01x12_Female, SW1 SW_Push, SW2 SW_Push, SW3 SW_Push

Commit message: Add protection diode for LCD
Parts:
- added D1: 1N4001, Diode_THT:D_DO-41_SOD81_P10.16mm_Horizontal, F.Cu at (84.6, 35.1)
- moved RV1 2.20 mm to (88.9, 39.8), turned to 270 degrees
Connections:
- J1 pad 1: Net-(C1-Pad1) -> Net-(D1-Pad2)
Routing:
- net Net-(DS1-Pad3): track 45.3 -> 21.8 mm
- net Net-(C1-Pad1): track 97.3 -> 119.8 mm, vias 4 -> 2
- net GND: track 246.4 -> 240.1 mm
- net Net-(D1-Pad2): track 0.00 -> 5.01 mm
